Commit message: Add right wheel

File: my_rb1_description/urdf/my_rb1_robot.xacro (robot description, xacro)
@@ -19,15 +19,15 @@
     <link name="base_link">
         <inertial>
+            <origin xyz="0 0 0.3" rpy="0 0 0" />
             <mass value="${base_m}" />
-            <origin xyz="0 0 0.3" rpy="0 0 0" />
             <!-- Ix = Iy = 1/12 * m * (3r^2 + h^2) -->
             <!-- Iz = 1/2 * m * r^2 -->
             <inertia
-                ixx="${(1/12) * base_m * (3 * base_r * base_r + base_h * base_h)}"
+                ixx="${(base_m / 12) * (3 * base_r*base_r + base_h * base_h)}"
                 ixy="0"
                 ixz="0"
-                iyy="${(1/12) * base_m * (3 * base_r * base_r + base_h * base_h)}"
+                iyy="${(base_m / 12) * (3 * base_r * base_r + base_h * base_h)}"
                 iyz="0"
-                izz="${0.5 * base_m * base_r * base_r}" />
+                izz="${(base_m / 2) * base_r * base_r}" />
         </inertial>
         <collision>
@@ -64,10 +64,48 @@
             <!-- Iz = 1/2 * m * r^2 -->
             <inertia
-                ixx="${(1/12) * wheel_m * (3 * wheel_r * wheel_r + wheel_h * wheel_h)}"
+                ixx="${(wheel_m / 12) * (3 * wheel_r * wheel_r + wheel_h * wheel_h)}"
                 ixy="0"
                 ixz="0"
-                iyy="${(1/12) * wheel_m * (3 * wheel_r * wheel_r + wheel_h * wheel_h)}"
+                iyy="${(wheel_m / 12) * (3 * wheel_r * wheel_r + wheel_h * wheel_h)}"
                 iyz="0"
-                izz="${0.5 * wheel_m * wheel_r * wheel_r}" />
+                izz="${(wheel_m / 2) * wheel_r * wheel_r}" />
+        </inertial>
+        <collision>
+            <origin xyz="0 0 0" rpy="${PI/2} 0 0" />
+            <geometry>
+                <cylinder length="${wheel_h}" radius="${wheel_r}"/>
+            </geometry>
+        </collision>
+        <visual>
+            <origin xyz="0 0 0" rpy="${PI/2} 0 0" />
+            <geometry>
+                <cylinder length="${wheel_h}" radius="${wheel_r}"/>
+            </geometry>
+            <material name="red" />
+        </visual>
+    </link>
+    <!-- Joint - base / right wheel -->
+    <joint name="base_to_right_wheel" type="continuous">
+        <origin rpy="0 0 0" xyz="0 0.2 -0.15" />
+        <parent link="base_link" />
+        <child link="right_wheel" />
+        <axis rpy="0 0 0" xyz="0 1 0" />
+        <limit effort="10000" velocity="1000" />
+        <joint_properties damping="1.0" friction="1.0" />
+    </joint>
+    <!-- Link - right wheel -->
+    <link name="right_wheel">
+        <inertial>
+            <mass value="${wheel_m}" />
+            <origin xyz="0 0 0" rpy="0 0 0" />
+            <!-- Ix = Iy = 1/12 * m * (3r^2 + h^2) -->
+            <!-- Iz = 1/2 * m * r^2 -->
+            <inertia
+                ixx="${(wheel_m / 12) * (3 * wheel_r * wheel_r + wheel_h * wheel_h)}"
+                ixy="0"
+                ixz="0"
+                iyy="${(wheel_m / 12) * (3 * wheel_r * wheel_r + wheel_h * wheel_h)}"
+                iyz="0"
+                izz="${(wheel_m / 2) * wheel_r * wheel_r}" />
         </inertial>
         <collision>

Commit message: Add front caster

File: my_rb1_description/urdf/my_rb1_robot.xacro (robot description, xacro)
@@ -8,6 +8,12 @@
         <color rgba="0 0 ${204/255} 1"/>
     </material>
+    <material name="DarkBlue">
+        <color rgba="${51/255} ${51/255} ${104/255} 1" />
+    </material>
     <material name="red">
         <color rgba="${204/255} 0 0 1"/>
+    </material>
+    <material name="Grey">
+        <color rgba="${153/255} ${153/255} ${153/255} 1" />
     </material>
     <!-- Constants -->
@@ -123,3 +129,58 @@
         </visual>
     </link>
+    <!-- Caster properties -->
+    <xacro:property name="caster_r" value="${0.025 / 2}" />
+    <xacro:property name="caster_m" value="1" />
+    <!-- Joint - base / left wheel -->
+    <joint name="base_to_front_caster" type="fixed">
+        <origin rpy="0 0 0" xyz="0.1 0 -0.15" />
+        <parent link="base_link" />
+        <child link="front_caster" />
+        <axis rpy="0 0 0" xyz="0 1 0" />
+        <limit effort="10000" velocity="1000" />
+        <joint_properties damping="1.0" friction="0" />
+    </joint>
+    <!-- Link - front caster -->
+    <link name="front_caster">
+        <inertial>
+            <mass value="${caster_m}" />
+            <origin xyz="0 0 0" rpy="0 0 0" />
+            <!-- Ix = Iy = Iz = 2/5 * m * r^2 -->
+            <inertia
+                ixx="${(2/5) * caster_m * caster_r * caster_r}"
+                ixy="0"
+                ixz="0"
+                iyy="${(2/5) * caster_m * caster_r * caster_r}"
+                iyz="0"
+                izz="${(2/5) * caster_m * caster_r * caster_r}" />
+        </inertial>
+        <!-- Caster wheel support -->
+        <collision>
+            <origin rpy="0 0 0" xyz="0 0 ${caster_r/2}" />
+            <geometry>
+                <sphere radius="${caster_r * 2}" />
+            </geometry>
+        </collision>
+        <visual>
+            <origin rpy="0 0 0" xyz="0 0 ${caster_r/2}" />
+            <geometry>
+                <sphere radius="${caster_r * 2}" />
+            </geometry>
+            <material name="DarkBlue" />
+        </visual>
+        <!-- Caster wheel -->
+        <collision>
+            <origin rpy="0 0 0" xyz="0 0 -${caster_r}" />
+            <geometry>
+                <sphere radius="${caster_r}" />
+            </geometry>
+        </collision>
+        <visual>
+            <origin rpy="0 0 0" xyz="0 0 -${caster_r}" />
+            <geometry>
+                <sphere radius="${caster_r}" />
+            </geometry>
+            <material name="Grey" />
+        </visual>
+    </link>
 </robot>

Commit message: Add back caster

File: my_rb1_description/urdf/my_rb1_robot.xacro (robot description, xacro)
@@ -50,5 +50,5 @@
     </link>
     <!-- Wheel properties -->
-    <xacro:property name="wheel_r" value="0.025" />
+    <xacro:property name="wheel_r" value="${0.05 / 2}" />
     <xacro:property name="wheel_h" value="0.025" />
     <xacro:property name="wheel_m" value="1" />
@@ -132,5 +132,5 @@
     <xacro:property name="caster_r" value="${0.025 / 2}" />
     <xacro:property name="caster_m" value="1" />
-    <!-- Joint - base / left wheel -->
+    <!-- Joint - base / front caster -->
     <joint name="base_to_front_caster" type="fixed">
         <origin rpy="0 0 0" xyz="0.1 0 -0.15" />
@@ -184,3 +184,55 @@
         </visual>
     </link>
+    <!-- Joint - base / back caster -->
+    <joint name="base_to_back_caster" type="fixed">
+        <origin rpy="0 0 0" xyz="-0.1 0 -0.15" />
+        <parent link="base_link" />
+        <child link="back_caster" />
+        <axis rpy="0 0 0" xyz="0 1 0" />
+        <limit effort="10000" velocity="1000" />
+        <joint_properties damping="1.0" friction="0" />
+    </joint>
+    <!-- Link - back caster -->
+    <link name="back_caster">
+        <inertial>
+            <mass value="${caster_m}" />
+            <origin xyz="0 0 0" rpy="0 0 0" />
+            <!-- Ix = Iy = Iz = 2/5 * m * r^2 -->
+            <inertia
+                ixx="${(2/5) * caster_m * caster_r * caster_r}"
+                ixy="0"
+                ixz="0"
+                iyy="${(2/5) * caster_m * caster_r * caster_r}"
+                iyz="0"
+                izz="${(2/5) * caster_m * caster_r * caster_r}" />
+        </inertial>
+        <!-- Caster wheel support -->
+        <collision>
+            <origin rpy="0 0 0" xyz="0 0 ${caster_r/2}" />
+            <geometry>
+                <sphere radius="${caster_r * 2}" />
+            </geometry>
+        </collision>
+        <visual>
+            <origin rpy="0 0 0" xyz="0 0 ${caster_r/2}" />
+            <geometry>
+                <sphere radius="${caster_r * 2}" />
+            </geometry>
+            <material name="DarkBlue" />
+        </visual>
+        <!-- Caster wheel -->
+        <collision>
+            <origin rpy="0 0 0" xyz="0 0 -${caster_r}" />
+            <geometry>
+                <sphere radius="${caster_r}" />
+            </geometry>
+        </collision>
+        <visual>
+            <origin rpy="0 0 0" xyz="0 0 -${caster_r}" />
+            <geometry>
+                <sphere radius="${caster_r}" />
+            </geometry>
+            <material name="Grey" />
+        </visual>
+    </link>
 </robot>

Commit message: Add base_footprint
- Add empty link: base_footprint
  - add joint connecting it to the base_link
- Replace 0.15 with ${base_h / 2}

File: my_rb1_description/urdf/my_rb1_robot.xacro (robot description, xacro)
@@ -25,10 +25,10 @@
     <link name="base_link">
         <inertial>
-            <origin xyz="0 0 0.3" rpy="0 0 0" />
+            <origin xyz="0 0 0" rpy="0 0 0" />
             <mass value="${base_m}" />
             <!-- Ix = Iy = 1/12 * m * (3r^2 + h^2) -->
             <!-- Iz = 1/2 * m * r^2 -->
             <inertia
-                ixx="${(base_m / 12) * (3 * base_r*base_r + base_h * base_h)}"
+                ixx="${(base_m / 12) * (3 * base_r * base_r + base_h * base_h)}"
                 ixy="0"
                 ixz="0"
@@ -49,4 +49,12 @@
         </visual>
     </link>
+    <!-- Joint - base / base_footprint -->
+    <joint name="base_to_base_footprint" type="fixed">
+        <origin rpy="0 0 0" xyz="0 0 -${base_h / 2}" />
+        <parent link="base_link" />
+        <child link="base_footprint" />
+    </joint>
+    <!-- Link - base_footprint -->
+    <link name="base_footprint" />
     <!-- Wheel properties -->
     <xacro:property name="wheel_r" value="${0.05 / 2}" />
@@ -55,5 +63,5 @@
     <!-- Joint - base / left wheel -->
     <joint name="base_to_left_wheel" type="continuous">
-        <origin rpy="0 0 0" xyz="0 -0.2 -0.15" />
+        <origin rpy="0 0 0" xyz="0 -0.2 -${base_h / 2}" />
         <parent link="base_link" />
         <child link="left_wheel" />
@@ -93,5 +101,5 @@
     <!-- Joint - base / right wheel -->
     <joint name="base_to_right_wheel" type="continuous">
-        <origin rpy="0 0 0" xyz="0 0.2 -0.15" />
+        <origin rpy="0 0 0" xyz="0 0.2 -${base_h / 2}" />
         <parent link="base_link" />
         <child link="right_wheel" />
@@ -134,5 +142,5 @@
     <!-- Joint - base / front caster -->
     <joint name="base_to_front_caster" type="fixed">
-        <origin rpy="0 0 0" xyz="0.1 0 -0.15" />
+        <origin rpy="0 0 0" xyz="0.1 0 -${base_h / 2}" />
         <parent link="base_link" />
         <child link="front_caster" />
@@ -186,5 +194,5 @@
     <!-- Joint - base / back caster -->
     <joint name="base_to_back_caster" type="fixed">
-        <origin rpy="0 0 0" xyz="-0.1 0 -0.15" />
+        <origin rpy="0 0 0" xyz="-0.1 0 -${base_h / 2}" />
         <parent link="base_link" />
         <child link="back_caster" />

Commit message: Add interia macros
- Add macro for calculating inertia for cylinders
- Add macro for calculating inertia for spheres
- Refactored to use macros for inertia in both wheels and both casters

File: my_rb1_description/urdf/my_rb1_robot.xacro (robot description, xacro)
@@ -19,4 +19,22 @@
     <!-- Constants -->
     <xacro:property name="PI" value="3.1415926535897931"/>
+    <!-- Macros -->
+    <xacro:macro name="cylinder_inertia" params="m r h">
+        <!-- Ix = Iy = 1/12 * m * (3r^2 + h^2) -->
+        <!-- Iz = 1/2 * m * r^2 -->
+        <inertia
+            ixx="${(m/12) * (3 * r*r + h*h)}" ixy = "0" ixz = "0"
+            iyy="${(m/12) * (3 * r*r + h*h)}" iyz = "0"
+            izz="${(m/2) * r*r}"
+        />
+    </xacro:macro>
+    <xacro:macro name="sphere_interia" params="m r">
+        <!-- Ix = Iy = Iz = 2/5 * m * r^2 -->
+        <inertia
+            ixx="${(2/5) * m * r*r}" ixy="0" ixz="0"
+            iyy="${(2/5) * m * r*r}" iyz="0"
+            izz="${(2/5) * m * r*r}"
+        />
+    </xacro:macro>
     <!-- Link - base -->
     <xacro:property name="base_r" value="0.25" />
@@ -27,13 +45,5 @@
             <origin xyz="0 0 0" rpy="0 0 0" />
             <mass value="${base_m}" />
-            <!-- Ix = Iy = 1/12 * m * (3r^2 + h^2) -->
-            <!-- Iz = 1/2 * m * r^2 -->
-            <inertia
-                ixx="${(base_m / 12) * (3 * base_r * base_r + base_h * base_h)}"
-                ixy="0"
-                ixz="0"
-                iyy="${(base_m / 12) * (3 * base_r * base_r + base_h * base_h)}"
-                iyz="0"
-                izz="${(base_m / 2) * base_r * base_r}" />
+            <xacro:cylinder_inertia m="${base_m}" r="${base_r}" h="${base_h}" />
         </inertial>
         <collision>
@@ -75,13 +85,5 @@
             <mass value="${wheel_m}" />
             <origin xyz="0 0 0" rpy="0 0 0" />
-            <!-- Ix = Iy = 1/12 * m * (3r^2 + h^2) -->
-            <!-- Iz = 1/2 * m * r^2 -->
-            <inertia
-                ixx="${(wheel_m / 12) * (3 * wheel_r * wheel_r + wheel_h * wheel_h)}"
-                ixy="0"
-                ixz="0"
-                iyy="${(wheel_m / 12) * (3 * wheel_r * wheel_r + wheel_h * wheel_h)}"
-                iyz="0"
-                izz="${(wheel_m / 2) * wheel_r * wheel_r}" />
+            <xacro:cylinder_inertia m="${wheel_m}" r="${wheel_r}" h="${wheel_h}" />
         </inertial>
         <collision>
@@ -113,13 +115,5 @@
             <mass value="${wheel_m}" />
             <origin xyz="0 0 0" rpy="0 0 0" />
-            <!-- Ix = Iy = 1/12 * m * (3r^2 + h^2) -->
-            <!-- Iz = 1/2 * m * r^2 -->
-            <inertia
-                ixx="${(wheel_m / 12) * (3 * wheel_r * wheel_r + wheel_h * wheel_h)}"
-                ixy="0"
-                ixz="0"
-                iyy="${(wheel_m / 12) * (3 * wheel_r * wheel_r + wheel_h * wheel_h)}"
-                iyz="0"
-                izz="${(wheel_m / 2) * wheel_r * wheel_r}" />
+            <xacro:cylinder_inertia m="${wheel_m}" r="${wheel_r}" h="${wheel_h}" />
         </inertial>
         <collision>
@@ -154,12 +148,5 @@
             <mass value="${caster_m}" />
             <origin xyz="0 0 0" rpy="0 0 0" />
-            <!-- Ix = Iy = Iz = 2/5 * m * r^2 -->
-            <inertia
-                ixx="${(2/5) * caster_m * caster_r * caster_r}"
-                ixy="0"
-                ixz="0"
-                iyy="${(2/5) * caster_m * caster_r * caster_r}"
-                iyz="0"
-                izz="${(2/5) * caster_m * caster_r * caster_r}" />
+            <xacro:sphere_interia m="${caster_m}" r="${caster_r}" />
         </inertial>
         <!-- Caster wheel support -->
@@ -206,12 +193,5 @@
             <mass value="${caster_m}" />
             <origin xyz="0 0 0" rpy="0 0 0" />
-            <!-- Ix = Iy = Iz = 2/5 * m * r^2 -->
-            <inertia
-                ixx="${(2/5) * caster_m * caster_r * caster_r}"
-                ixy="0"
-                ixz="0"
-                iyy="${(2/5) * caster_m * caster_r * caster_r}"
-                iyz="0"
-                izz="${(2/5) * caster_m * caster_r * caster_r}" />
+            <xacro:sphere_interia m="${caster_m}" r="${caster_r}" />
         </inertial>
         <!-- Caster wheel support -->

Commit message: Add front laser
- Modeled after the Hokuyo UBG-04LX-F01
  - https://www.hokuyo-aut.jp/search/single.php?serial=164
- Add front_laser link and joint connecting it to base_link
- Add box_inertia macro to calculate the inertia of a box

File: my_rb1_description/urdf/my_rb1_robot.xacro (robot description, xacro)
@@ -8,5 +8,5 @@
         <color rgba="0 0 ${204/255} 1"/>
     </material>
-    <material name="DarkBlue">
+    <material name="dark_blue">
         <color rgba="${51/255} ${51/255} ${104/255} 1" />
     </material>
@@ -14,6 +14,9 @@
         <color rgba="${204/255} 0 0 1"/>
     </material>
-    <material name="Grey">
+    <material name="grey">
         <color rgba="${153/255} ${153/255} ${153/255} 1" />
+    </material>
+    <material name="dark_grey">
+        <color rgba="${45/255} ${45/255} ${45/255} 1" />
     </material>
     <!-- Constants -->
@@ -21,6 +24,4 @@
     <!-- Macros -->
     <xacro:macro name="cylinder_inertia" params="m r h">
-        <!-- Ix = Iy = 1/12 * m * (3r^2 + h^2) -->
-        <!-- Iz = 1/2 * m * r^2 -->
         <inertia
             ixx="${(m/12) * (3 * r*r + h*h)}" ixy = "0" ixz = "0"
@@ -30,5 +31,4 @@
     </xacro:macro>
     <xacro:macro name="sphere_interia" params="m r">
-        <!-- Ix = Iy = Iz = 2/5 * m * r^2 -->
         <inertia
             ixx="${(2/5) * m * r*r}" ixy="0" ixz="0"
@@ -37,8 +37,15 @@
         />
     </xacro:macro>
+    <xacro:macro name="box_inertia" params="m x y z">
+        <inertia
+            ixx="${(m/12) * (x*x + z*z)}" ixy="0" ixz="0"
+            iyy="${(m/12) * (y*y + x*x)}" iyz="0"
+            izz="${(m/12) * (y*y + z*z)}"
+        />
+    </xacro:macro>
     <!-- Link - base -->
     <xacro:property name="base_r" value="0.25" />
     <xacro:property name="base_h" value="0.30" />
-    <xacro:property name="base_m" value="20" />
+    <xacro:property name="base_m" value="20.74" />
     <link name="base_link">
         <inertial>
@@ -162,5 +169,5 @@
                 <sphere radius="${caster_r * 2}" />
             </geometry>
-            <material name="DarkBlue" />
+            <material name="dark_blue" />
         </visual>
         <!-- Caster wheel -->
@@ -176,5 +183,5 @@
                 <sphere radius="${caster_r}" />
             </geometry>
-            <material name="Grey" />
+            <material name="grey" />
         </visual>
     </link>
@@ -207,5 +214,5 @@
                 <sphere radius="${caster_r * 2}" />
             </geometry>
-            <material name="DarkBlue" />
+            <material name="dark_blue" />
         </visual>
         <!-- Caster wheel -->
@@ -221,5 +228,39 @@
                 <sphere radius="${caster_r}" />
             </geometry>
-            <material name="Grey" />
+            <material name="grey" />
+        </visual>
+    </link>
+    <!-- Laser properties -->
+    <xacro:property name="laser_x" value="${75.0 / 1000}" />
+    <xacro:property name="laser_y" value="${60.0 / 1000}" />
+    <xacro:property name="laser_z" value="${60.0 / 1000}" />
+    <xacro:property name="laser_m" value="${260.0 / 1000}" />
+    <!-- Joint - base / front laser -->
+    <joint name="base_to_front_laser" type="fixed">
+        <!-- rotate the laser by 180 degrees -->
+        <origin rpy="${PI} 0 0" xyz="${base_r} 0 ${base_h / 4}" />
+        <parent link="base_link" />
+        <child link="front_laser" />
+    </joint>
+    <!-- Link - front laser -->
+    <!-- Modeled after a Hokuyo UBG-04LX-F01 -->
+    <link name="front_laser">
+        <inertial>
+            <mass value="${laser_m}" />
+            <origin xyz="0 0 0" rpy="0 0 0" />
+            <xacro:box_inertia m="${laser_m}" x="${laser_x}" y="${laser_y}" z="${laser_z}" />
+        </inertial>
+        <collision>
+            <origin xyz="0 0 0" rpy="0 0 0" />
+            <geometry>
+                <box size="${laser_x} ${laser_y}  ${laser_z}" />
+            </geometry>
+        </collision>
+        <visual>
+            <origin xyz="0 0 0" rpy="0 0 0" />
+            <geometry>
+                <box size="${laser_x} ${laser_y}  ${laser_z}" />
+            </geometry>
+            <material name="dark_grey" />
         </visual>
     </link>

Commit message: Set base color to black and position robot in square

File: my_rb1_description/urdf/my_rb1_robot.xacro (robot description, xacro)
@@ -4,4 +4,8 @@
     <xacro:include filename="$(find robot_description)/urdf/robot.gazebo" />
     -->
+    <!-- Gazebo -->
+    <gazebo reference="base_link">
+        <material>Gazebo/Black</material>
+    </gazebo>
     <!-- Materials -->
     <material name="blue">

Commit message: Add differential drive to robot
- Add xacro parameter for the base_to_wheel_offset in the y-axis
- Move the gazebo tags to the end of the file so they can use the xacro
parameters
- Add the differential_drive_controller
  - separation = base_to_wheel_offset_y * 2
  - diameter = wheel_r * 2
- Add mu1 and mu2 to gazebo references for the wheels and casters
- Add preserveFixedJoint(true) to the caster references

File: my_rb1_description/urdf/my_rb1_robot.xacro (robot description, xacro)
@@ -4,8 +4,4 @@
     <xacro:include filename="$(find robot_description)/urdf/robot.gazebo" />
     -->
-    <!-- Gazebo -->
-    <gazebo reference="base_link">
-        <material>Gazebo/Black</material>
-    </gazebo>
     <!-- Materials -->
     <material name="blue">
@@ -79,4 +75,5 @@
     <link name="base_footprint" />
     <!-- Wheel properties -->
+    <xacro:property name="base_to_wheel_offset_y" value="0.2" />
     <xacro:property name="wheel_r" value="${0.05 / 2}" />
     <xacro:property name="wheel_h" value="0.025" />
@@ -84,5 +81,5 @@
     <!-- Joint - base / left wheel -->
     <joint name="base_to_left_wheel" type="continuous">
-        <origin rpy="0 0 0" xyz="0 -0.2 -${base_h / 2}" />
+        <origin rpy="0 0 0" xyz="0 ${base_to_wheel_offset_y} -${base_h / 2}" />
         <parent link="base_link" />
         <child link="left_wheel" />
@@ -114,5 +111,5 @@
     <!-- Joint - base / right wheel -->
     <joint name="base_to_right_wheel" type="continuous">
-        <origin rpy="0 0 0" xyz="0 0.2 -${base_h / 2}" />
+        <origin rpy="0 0 0" xyz="0 -${base_to_wheel_offset_y} -${base_h / 2}" />
         <parent link="base_link" />
         <child link="right_wheel" />
@@ -269,3 +266,40 @@
         </visual>
     </link>
+    <!-- Gazebo -->
+    <gazebo reference="base_link">
+        <material>Gazebo/Black</material>
+    </gazebo>
+    <gazebo reference="base_to_left_wheel">
+        <mu1>1</mu1>
+        <mu2>1</mu2>
+    </gazebo>
+    <gazebo reference="base_to_right_wheel">
+        <mu1>1</mu1>
+        <mu2>1</mu2>
+    </gazebo>
+    <gazebo reference="base_to_front_caster">
+        <preserveFixedJoint>true</preserveFixedJoint>
+        <mu1>0</mu1>
+        <mu2>0</mu2>
+    </gazebo>
+    <gazebo reference="base_to_back_caster">
+        <preserveFixedJoint>true</preserveFixedJoint>
+        <mu1>0</mu1>
+        <mu2>0</mu2>
+    </gazebo>
+    <gazebo>
+        <plugin filename="libgazebo_ros_diff_drive.so" name="differential_drive_controller">
+            <alwaysOn>true</alwaysOn>
+            <updateRate>20</updateRate>
+            <leftJoint>base_to_left_wheel</leftJoint>
+            <rightJoint>base_to_right_wheel</rightJoint>
+            <wheelSeparation>${base_to_wheel_offset_y * 2}</wheelSeparation>
+            <wheelDiameter>${wheel_r * 2}</wheelDiameter>
+            <torque>10</torque>
+            <commandTopic>cmd_vel</commandTopic>
+            <odometryTopic>odom</odometryTopic>
+            <odometryFrame>odom</odometryFrame>
+            <robotBaseFrame>base_link</robotBaseFrame>
+        </plugin>
+    </gazebo>
 </robot>
