Commit message: Add laser
- robot is turning to the left and wobbling
  - increades wheel length to 0.3 to try to fix
  - still happening
TODO: check height of caster/wheels

File: my_rb1_description/urdf/my_rb1_robot.xacro (robot description, xacro)
@@ -77,5 +77,5 @@
     <xacro:property name="base_to_wheel_offset_y" value="0.2" />
     <xacro:property name="wheel_r" value="${0.05 / 2}" />
-    <xacro:property name="wheel_h" value="0.025" />
+    <xacro:property name="wheel_h" value="0.03" />
     <xacro:property name="wheel_m" value="1" />
     <!-- Joint - base / left wheel -->
@@ -266,5 +266,5 @@
         </visual>
     </link>
-    <!-- Gazebo -->
+    <!-- Gazebo tags -->
     <gazebo reference="base_link">
         <material>Gazebo/Black</material>
@@ -287,4 +287,7 @@
         <mu1>0</mu1>
         <mu2>0</mu2>
+    </gazebo>
+    <gazebo reference="base_to_front_laser">
+        <preserveFixedJoint>true</preserveFixedJoint>
     </gazebo>
     <gazebo>
@@ -303,3 +306,34 @@
         </plugin>
     </gazebo>
+    <gazebo reference="front_laser">
+        <sensor type="ray" name="head_hokuyo_sensor">
+            <pose>0 0 0 0 0 0</pose>
+            <visualize>false</visualize>
+            <update_rate>20</update_rate>
+            <ray>
+                <scan>
+                    <horizontal>
+                        <samples>720</samples>
+                        <resolution>1</resolution>
+                        <min_angle>-1.570796</min_angle>
+                        <max_angle>1.570796</max_angle>
+                    </horizontal>
+                </scan>
+                <range>
+                    <min>0.20</min>
+                    <max>10.0</max>
+                    <resolution>0.01</resolution>
+                </range>
+                <noise>
+                    <type>gaussian</type>
+                    <mean>0.0</mean>
+                    <stddev>0.01</stddev>
+                </noise>
+            </ray>
+            <plugin name="gazebo_ros_head_hokuyo_controller" filename="libgazebo_ros_laser.so">
+                <topicName>/scan</topicName>
+                <frameName>sensor_laser</frameName>
+            </plugin>
+        </sensor>
+    </gazebo>
 </robot>

Commit message: Fixed turning issue
- I had the <mu1> and <mu2> tags on the base_to_xxx joints instead of on
the actual links
- Moving them corrected the issue

File: my_rb1_description/urdf/my_rb1_robot.xacro (robot description, xacro)
@@ -47,5 +47,5 @@
     <xacro:property name="base_r" value="0.25" />
     <xacro:property name="base_h" value="0.30" />
-    <xacro:property name="base_m" value="20.74" />
+    <xacro:property name="base_m" value="17.74" />
     <link name="base_link">
         <inertial>
@@ -78,5 +78,5 @@
     <xacro:property name="wheel_r" value="${0.05 / 2}" />
     <xacro:property name="wheel_h" value="0.03" />
-    <xacro:property name="wheel_m" value="1" />
+    <xacro:property name="wheel_m" value="2" />
     <!-- Joint - base / left wheel -->
     <joint name="base_to_left_wheel" type="continuous">
@@ -141,5 +141,5 @@
     <!-- Caster properties -->
     <xacro:property name="caster_r" value="${0.025 / 2}" />
-    <xacro:property name="caster_m" value="1" />
+    <xacro:property name="caster_m" value="1.5" />
     <!-- Joint - base / front caster -->
     <joint name="base_to_front_caster" type="fixed">
@@ -155,5 +155,5 @@
         <inertial>
             <mass value="${caster_m}" />
-            <origin xyz="0 0 0" rpy="0 0 0" />
+            <origin xyz="0 0 -${caster_r}" rpy="0 0 0" />
             <xacro:sphere_interia m="${caster_m}" r="${caster_r}" />
         </inertial>
@@ -200,5 +200,5 @@
         <inertial>
             <mass value="${caster_m}" />
-            <origin xyz="0 0 0" rpy="0 0 0" />
+            <origin xyz="0 0 -${caster_r}" rpy="0 0 0" />
             <xacro:sphere_interia m="${caster_m}" r="${caster_r}" />
         </inertial>
@@ -270,21 +270,25 @@
         <material>Gazebo/Black</material>
     </gazebo>
-    <gazebo reference="base_to_left_wheel">
+    <gazebo reference="left_wheel">
         <mu1>1</mu1>
         <mu2>1</mu2>
     </gazebo>
-    <gazebo reference="base_to_right_wheel">
+    <gazebo reference="right_wheel">
         <mu1>1</mu1>
         <mu2>1</mu2>
     </gazebo>
+    <gazebo reference="front_caster">
+        <mu1>0</mu1>
+        <mu2>0</mu2>
+    </gazebo>
+    <gazebo reference="back_caster">
+        <mu1>0</mu1>
+        <mu2>0</mu2>
+    </gazebo>
     <gazebo reference="base_to_front_caster">
         <preserveFixedJoint>true</preserveFixedJoint>
-        <mu1>0</mu1>
-        <mu2>0</mu2>
     </gazebo>
     <gazebo reference="base_to_back_caster">
         <preserveFixedJoint>true</preserveFixedJoint>
-        <mu1>0</mu1>
-        <mu2>0</mu2>
     </gazebo>
     <gazebo reference="base_to_front_laser">
@@ -309,5 +313,5 @@
         <sensor type="ray" name="head_hokuyo_sensor">
             <pose>0 0 0 0 0 0</pose>
-            <visualize>true</visualize>
+            <visualize>false</visualize>
             <update_rate>20</update_rate>
             <ray>
